File: MP3_board_first/mp3.sch (EAGLE design)
At the start: 17 parts, among them U1 ATMEGA328P_PDIP_OM

Commit message: first soldered version of board
Parts:
- removed S6: MOMENTARY-SWITCH-SPST-PTH-RIGHT-ANGLE, SparkFun-Switches:MOMENTARY-SWITCH-SPST-PTH-RIGHT-ANGLE
- removed S7: MOMENTARY-SWITCH-SPST-PTH-6.0MM, SparkFun-Switches:MOMENTARY-SWITCH-SPST-PTH-6.0MM
- added J1, J2, J3: (no value), SparkFun-Connectors:CONN_01PTH_NO_SILK_KIT
- C1: device SparkFun-Capacitors:0.1UF-KIT-EZ-50V-20% -> christy:0.1UF-KIT-EZ-50V-20%
- U$1: device DFPlayer_v1:DFPLAYER -> christy:DFPLAYER
Connections:
- new net 3.3V: J3.1, U$1.GND_1
- new net N$8: J1.1, U$1.DAC_R
- new net N$9: J2.1, U$1.DAC_L
- net GND: no longer U$1.GND_1
- net N$5: now also U1.PB2(SS/OC1B); no longer U1.PB4(MISO)
- net NXF: now also U1.PB0(ICP)
- net PXF: now also U1.PD4(XCK/T0)
- net V_BATT: now also U1.AVCC; no longer U1.VCC
Other:
- moved on the sheet: R4
